File: passive-4x4/matrixmixer.kicad_pcb (KiCad board)
At the start: 2 copper layers, 100 x 100 mm, 58 parts, among them J1 Input 1, J2 Input 2, J3 Input 3, J4 Input 4, J5 Output 1, J6 Output 2, J7 Output 4, J8 Output 4, P1 Stereo/Sync, P10 EXT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

Commit message: Passive 4x4 v0.2
Connections:
- J1 pad 4: (no net) -> Net-(J1-Pad4)
- J1 pad 5: (no net) -> Net-(J1-Pad5)
- J2 pad 4: (no net) -> Net-(J2-Pad4)
- J2 pad 5: (no net) -> Net-(J2-Pad5)
- J3 pad 4: (no net) -> Net-(J3-Pad4)
- J3 pad 5: (no net) -> Net-(J3-Pad5)
- J4 pad 4: (no net) -> Net-(J4-Pad4)
- J4 pad 5: (no net) -> Net-(J4-Pad5)
- J5 pad 4: (no net) -> Net-(J5-Pad4)
- J5 pad 5: (no net) -> Net-(J5-Pad5)
- J6 pad 4: (no net) -> Net-(J6-Pad4)
- J6 pad 5: (no net) -> Net-(J6-Pad5)
- J7 pad 4: (no net) -> Net-(J7-Pad4)
- J7 pad 5: (no net) -> Net-(J7-Pad5)
- J8 pad 4: (no net) -> Net-(J8-Pad4)
- J8 pad 5: (no net) -> Net-(J8-Pad5)
- RV1 pad 1: in1 -> GND
- RV1 pad 3: GND -> in1
- RV10 pad 1: in2 -> GND
- RV10 pad 3: GND -> in2
- RV11 pad 1: in3 -> GND
- RV11 pad 3: GND -> in3
- RV12 pad 1: in4 -> GND
- RV12 pad 3: GND -> in4
- RV13 pad 1: in1 -> GND
- RV13 pad 3: GND -> in1
- RV14 pad 1: in2 -> GND
- RV14 pad 3: GND -> in2
- RV15 pad 1: in3 -> GND
- RV15 pad 3: GND -> in3
- RV16 pad 1: in4 -> GND
- RV16 pad 3: GND -> in4
- RV2 pad 1: in2 -> GND
- RV2 pad 3: GND -> in2
- RV3 pad 1: in3 -> GND
- RV3 pad 3: GND -> in3
- RV4 pad 1: in4 -> GND
- RV4 pad 3: GND -> in4
- RV5 pad 1: in1 -> GND
- RV5 pad 3: GND -> in1
- RV6 pad 1: in2 -> GND
- RV6 pad 3: GND -> in2
- RV7 pad 1: in3 -> GND
- RV7 pad 3: GND -> in3
- RV8 pad 1: in4 -> GND
- RV8 pad 3: GND -> in4
- RV9 pad 1: in1 -> GND
- RV9 pad 3: GND -> in1
Routing:
- net in2: track 87.0 -> 88.1 mm
- net in3: track 87.0 -> 88.1 mm
- net in4: track 87.0 -> 88.1 mm
- net GND: track 0.00 -> 0.64 mm
- added copper zone on F.Cu, net GND
Other:
- rule pad_to_mask_clearance: 0.2 -> 0
- board text added: "MatrixMix 4x4 v0.2 - design by MakerVan Labs Licensed under CC BY-SA 4.0 wiki.makervan.de/wiki/MatrixMix"
- board text removed: "MatrixMix 4x4 v0.1 - design by MakerVan Labs Licensed under CC BY-SA 4.0 wiki.makervan.de/wiki/MatrixMix"
