File: passive-4x4/matrixmixer.sch (KiCad schematic (older format))
At the start: 50 parts, among them J1 Input 1, J2 Input 2, J3 Input 3, J4 Input 4, J5 Output 1, J6 Output 2, J7 Output 4, J8 Output 4, P1 Stereo/Sync, P10 EXT, P2 Stereo/Sync, P3 Stereo/Sync, P4 Stereo/Sync, P5 Stereo/Sync, P6 Stereo/Sync, P7 Stereo/Sync, P8 Stereo/Sync, P9 EXT

Commit message: Passive 4x4 v0.2
Parts:
- J1, J2, J3, J4, J5, J6, J7, J8: symbol Jack_3.5mm_5pin -> w_connectors:Jack_3.5mm_5pin
- P1, P2, P3, P4, P5, P6, P7, P8: symbol CONN_01X03 -> matrixmixer-rescue:CONN_01X03
- P10, P9: symbol CONN_02X05 -> matrixmixer-rescue:CONN_02X05
- R1, R10, R11, R12, R13, R14, R15, R16, R2, R3, R4, R5, R6, R7, R8, R9: symbol R -> Device:R
- RV1, RV10, RV11, RV12, RV13, RV14, RV15, RV16, RV2, RV3, RV4, RV5, RV6, RV7, RV8, RV9: symbol POT -> matrixmixer-rescue:POT
Connections:
- net GND: now also RV1.1, RV10.1, RV11.1, RV12.1, RV13.1, RV14.1, RV15.1, RV16.1, RV2.1, RV3.1, RV4.1, RV5.1, RV6.1, RV7.1, RV8.1, RV9.1; no longer RV1.3, RV10.3, RV11.3, RV12.3, RV13.3, RV14.3, RV15.3, RV16.3, RV2.3, RV3.3, RV4.3, RV5.3, RV6.3, RV7.3, RV8.3, RV9.3
- net in1: now also RV1.3, RV13.3, RV5.3, RV9.3; no longer RV1.1, RV13.1, RV5.1, RV9.1
- net in2: now also RV10.3, RV14.3, RV2.3, RV6.3; no longer RV10.1, RV14.1, RV2.1, RV6.1
- net in3: now also RV11.3, RV15.3, RV3.3, RV7.3; no longer RV11.1, RV15.1, RV3.1, RV7.1
- net in4: now also RV12.3, RV16.3, RV4.3, RV8.3; no longer RV12.1, RV16.1, RV4.1, RV8.1
